Commit message: sonic_fusion node init

File: src/sonic_description/urdf/sonar_sensor.xacro (robot description, xacro)
@@ -2,5 +2,5 @@
 <robot xmlns:xacro="http://ros.org/wiki/xacro">
     <!-- MECCANUM WHEEL -->
-    <xacro:macro name="sonar_sensor" params="id parent origin rpy">
+    <xacro:macro name="sonar_sensor" params="id parent origin rpy fov">
     <!-- ULTRASONIC SENSORS -->
     <joint name="sensor_joint_${id}" type="fixed">
@@ -35,17 +35,17 @@
     <!-- USS Plugin -->
     <gazebo reference="uss_link_${id}">
-        <sensor type="ray" name="range_sensor_${id}">
+        <sensor type="lidar" name="range_sensor_${id}">
         <visualize>true</visualize>
         <ray>
             <scan>
             <horizontal>
-                <samples>1</samples>
-                <resolution>45</resolution>
-                <min_angle>-0.6545</min_angle>
-                <max_angle>0.6545</max_angle>
+                <samples>30</samples>
+                <resolution>1</resolution>
+                <min_angle>${-(fov/2)/180*PI}</min_angle>
+                <max_angle>${(fov/2)/180*PI}</max_angle>
             </horizontal>
             <vertical>
-                <samples>1</samples>
-                <resolution>15</resolution>
+                <samples>15</samples>
+                <resolution>1</resolution>
                 <min_angle>-0.04</min_angle>
                 <max_angle>0.04</max_angle>

File: src/sonic_description/urdf/sonic.gazebo.xacro (robot description, xacro)
@@ -43,5 +43,5 @@
       <publish_rate>40</publish_rate>
       <!-- Set if odom required -->
-      <publish_odom>false</publish_odom>
+      <publish_odom>true</publish_odom>
       <publish_odom_tf>false</publish_odom_tf>
       <!-- Frame IDs -->

File: src/sonic_description/urdf/sonic.urdf.xacro (robot description, xacro)
@@ -56,32 +56,32 @@
   <!-- SENSORS FRONT (id=FXX) -->
   <xacro:sonar_sensor id="F48" parent="base_link"
-  origin="${[body_length/2, 0.24, 0]}" rpy="0 0 ${PI/9}"/>
+  origin="${[body_length/2, 0.24, 0]}" rpy="0 0 ${PI/9}" fov="35"/>
   <xacro:sonar_sensor id="F49" parent="base_link"
-  origin="${[body_length/2, 0.12, 0]}" rpy="0 0 ${PI/18}"/>
+  origin="${[body_length/2, 0.12, 0]}" rpy="0 0 ${PI/18}" fov="35"/>
   <xacro:sonar_sensor id="F50" parent="base_link"
-  origin="${[body_length/2, 0, 0]}" rpy="0 0 0"/>
+  origin="${[body_length/2, 0, 0]}" rpy="0 0 0" fov="35"/>
   <xacro:sonar_sensor id="F51" parent="base_link"
-  origin="${[body_length/2, -0.12, 0]}" rpy="0 0 -${PI/18}"/>
+  origin="${[body_length/2, -0.12, 0]}" rpy="0 0 -${PI/18}" fov="35"/>
   <xacro:sonar_sensor id="F52" parent="base_link"
-  origin="${[body_length/2, -0.24, 0]}" rpy="0 0 -${PI/9}"/>
+  origin="${[body_length/2, -0.24, 0]}" rpy="0 0 -${PI/9}" fov="35"/>
   <!-- SENSORS REAR(id=RXX) -->
   <!--<xacro:sonar_sensor id="R48" parent="base_link"
-  origin="${[-body_length/2, 0.24, 0]}" rpy="0 0 ${PI - PI/9}"/>
+  origin="${[-body_length/2, 0.24, 0]}" rpy="0 0 ${PI - PI/9}" fov="35"/>
   <xacro:sonar_sensor id="R49" parent="base_link"
-  origin="${[-body_length/2, 0.12, 0]}" rpy="0 0 ${PI - PI/18}"/>
+  origin="${[-body_length/2, 0.12, 0]}" rpy="0 0 ${PI - PI/18}" fov="35"/>
   <xacro:sonar_sensor id="R50" parent="base_link"
-  origin="${[-body_length/2, 0, 0]}" rpy="0 0 ${PI}"/>
+  origin="${[-body_length/2, 0, 0]}" rpy="0 0 ${PI}" fov="35"/>
   <xacro:sonar_sensor id="R51" parent="base_link"
-  origin="${[-body_length/2, -0.12, 0]}" rpy="0 0 ${PI + PI/18}"/>
+  origin="${[-body_length/2, -0.12, 0]}" rpy="0 0 ${PI + PI/18}" fov="35"/>
   <xacro:sonar_sensor id="R52" parent="base_link"
-  origin="${[-body_length/2, -0.24, 0]}" rpy="0 0 ${PI + PI/9}"/>-->
+  origin="${[-body_length/2, -0.24, 0]}" rpy="0 0 ${PI + PI/9}" fov="35"/>-->
   <!-- SENSORS CHEEK (id=CXX) -->
   <!--<xacro:sonar_sensor id="C52" parent="base_link"
-  origin="${[-body_length/2+0.077, 0.42, 0]}" rpy="0 0 ${3*PI/4}"/>-->
+  origin="${[-body_length/2+0.077, 0.42, 0]}" rpy="0 0 ${3*PI/4}" fov="35"/>-->
   <xacro:sonar_sensor id="C51" parent="base_link"
-  origin="${[body_length/2-0.077, 0.42, 0]}" rpy="0 0 ${PI/4}"/>
+  origin="${[body_length/2-0.077, 0.42, 0]}" rpy="0 0 ${PI/4}" fov="35"/>
   <xacro:sonar_sensor id="C49" parent="base_link"
-  origin="${[body_length/2-0.077, -0.42, 0]}" rpy="0 0 ${-PI/4}"/>
+  origin="${[body_length/2-0.077, -0.42, 0]}" rpy="0 0 ${-PI/4}" fov="35"/>
   <!--<xacro:sonar_sensor id="C48" parent="base_link"
-  origin="${[-body_length/2+0.077, -0.42, 0]}" rpy="0 0 ${-3*PI/4}"/>-->
+  origin="${[-body_length/2+0.077, -0.42, 0]}" rpy="0 0 ${-3*PI/4}" fov="35"/>-->
 </robot>

Commit message: up to proba_map, fixed empty geom bug, first vis

File: src/sonic_description/urdf/sonar_sensor.xacro (robot description, xacro)
@@ -75,5 +75,5 @@
             <output_type>sensor_msgs/Range</output_type>
             <radiation_type>ultrasound</radiation_type>
-            <!-- <frame_name> ommited, will default to range_link -->
+            <frame_name>uss_link_${id}</frame_name>
         </plugin>
         </sensor>

File: src/sonic_description/urdf/sonic.urdf.xacro (robot description, xacro)
@@ -27,5 +27,5 @@
         <mesh filename="package://sonic_description/meshes/sonic_base.stl" scale="0.1 0.1 0.1"/>
       </geometry>
-      <material name="yellow" />
+      <material name="dark_grey" />
     </visual>
     <collision>
